File: Electronics/Ring Machine.sch (EAGLE design)
At the start: 19 parts, among them IC1 REG1117, U3 LM3480-3.3, X1 22-23-2081, X2 22-23-2081

Commit message: 5v regulator electronics
Connections:
- net GND: no longer R6.1, R6.2
- net VCC: now also R6.1, R6.2
Changed lines of the file:
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@@
 <part name="P+9" library="FAB_Hello" deviceset="VCC" device=""/>
 <part name="R6" library="ng" deviceset="RESISTOR" device="1206" value="0"/>
-<part name="GND18" library="FAB_Hello" deviceset="GND" device=""/>
-<part name="GND19" library="FAB_Hello" deviceset="GND" device=""/>
 <part name="R7" library="ng" deviceset="RESISTOR" device="1206" value="0"/>
 <part name="X1" library="con-molex" deviceset="22-23-2081" device=""/>
@@
 <part name="P+8" library="FAB_Hello" deviceset="VCC" device=""/>
 <part name="GND6" library="FAB_Hello" deviceset="GND" device=""/>
+<part name="P+10" library="FAB_Hello" deviceset="VCC" device=""/>
+<part name="P+11" library="FAB_Hello" deviceset="VCC" device=""/>
 </parts>
 <sheets>
@@
 <instance part="P+9" gate="VCC" x="76.2" y="-5.08" rot="R90"/>
 <instance part="R6" gate="G$1" x="83.82" y="-15.24"/>
-<instance part="GND18" gate="1" x="91.44" y="-15.24" rot="R90"/>
-<instance part="GND19" gate="1" x="76.2" y="-15.24" rot="R270"/>
 <instance part="R7" gate="G$1" x="139.7" y="45.72"/>
 <instance part="X1" gate="-1" x="129.54" y="12.7"/>
@@
 <instance part="P+8" gate="VCC" x="-12.7" y="91.44" rot="R90"/>
 <instance part="GND6" gate="1" x="10.16" y="76.2" rot="R90"/>
+<instance part="P+10" gate="VCC" x="76.2" y="-15.24" rot="R90"/>
+<instance part="P+11" gate="VCC" x="91.44" y="-15.24" rot="R270"/>
 </instances>
 <busses>
@@
 <pinref part="JP5" gate="-2" pin="1"/>
 <pinref part="GND13" gate="1" pin="GND"/>
-</segment>
-<segment>
-<pinref part="R6" gate="G$1" pin="2"/>
-<pinref part="GND18" gate="1" pin="GND"/>
-</segment>
-<segment>
-<pinref part="R6" gate="G$1" pin="1"/>
-<pinref part="GND19" gate="1" pin="GND"/>
 </segment>
 <segment>
@@
 <pinref part="P+8" gate="VCC" pin="VCC"/>
 </segment>
-</net>
+<segment>
+<pinref part="R6" gate="G$1" pin="1"/>
+<pinref part="P+10" gate="VCC" pin="VCC"/>
+</segment>
+<segment>
+<pinref part="R6" gate="G$1" pin="2"/>
+<pinref part="P+11" gate="VCC" pin="VCC"/>
+</segment>
+</net>
